File: stemthortyto/stemthortyto.kicad_pcb (KiCad board)
At the start: 8 copper layers, 88.7 x 29.2 mm, 66 parts, among them IC1 E22-900M22S, J1 Jack-DC, Q1 BCV29, U1 LT1585-3.3, U2 ADXL343, U3 RK3588S, U4 K4UCE3Q4AB-MGCL, U5 FEMDRW032G-88A19

Commit message: Add files via upload
Parts:
- added C12: 0.1μf, Capacitor_SMD:C_0201_0603Metric, B.Cu at (84.5, 65.8)
- added C12: 0.1μf, Capacitor_SMD:C_0201_0603Metric, B.Cu at (87.8, 76.2)
- added C12: 0.1μf, Capacitor_SMD:C_0201_0603Metric, B.Cu at (86.3, 74.8)
- added C12: 0.1μf, Capacitor_SMD:C_0201_0603Metric, B.Cu at (87.7, 65.6)
- added C12: 0.1μf, Capacitor_SMD:C_0201_0603Metric, B.Cu at (80.6, 67.7)
- added C12: 0.1μf, Capacitor_SMD:C_0201_0603Metric, B.Cu at (86.1, 67.7)
- added C18: 0.1μf, Capacitor_SMD:C_0201_0603Metric, B.Cu at (81.7, 64.2)
- added C21: 0.1μf, Capacitor_SMD:C_0201_0603Metric, B.Cu at (85.4, 63.7)
- added C21: 0.1μf, Capacitor_SMD:C_0201_0603Metric, B.Cu at (84.7, 68.8)
- added C21: 0.1μf, Capacitor_SMD:C_0201_0603Metric, B.Cu at (84.4, 67.0)
- added C23: 0.1μf, Capacitor_SMD:C_0201_0603Metric, B.Cu at (87.7, 68.4)
- added C24: 0.1μf, Capacitor_SMD:C_0201_0603Metric, B.Cu at (81.9, 72.9)
- added C25: 0.1μf, Capacitor_SMD:C_0201_0603Metric, B.Cu at (83.9, 72.8)
- added C25: 0.1μf, Capacitor_SMD:C_0201_0603Metric, B.Cu at (87.9, 72.9)
- added C25: 0.1μf, Capacitor_SMD:C_0201_0603Metric, B.Cu at (82.0, 68.9)
- added C25: 0.1μf, Capacitor_SMD:C_0201_0603Metric, B.Cu at (79.0, 72.9)
- added C25: 0.1μf, Capacitor_SMD:C_0201_0603Metric, B.Cu at (83.9, 74.1)
- added C25: 0.1μf, Capacitor_SMD:C_0201_0603Metric, B.Cu at (82.9, 74.4)
- added C31: 0.1μf, Capacitor_SMD:C_0201_0603Metric, B.Cu at (81.8, 68.0)
- added C31: 0.1μf, Capacitor_SMD:C_0201_0603Metric, B.Cu at (87.7, 67.0)
- added C31: 0.1μf, Capacitor_SMD:C_0201_0603Metric, B.Cu at (85.0, 68.0)
- added C31: 0.1μf, Capacitor_SMD:C_0201_0603Metric, B.Cu at (79.0, 67.0)
- added C44: 0.1μf, Capacitor_SMD:C_0201_0603Metric, B.Cu at (82.2, 65.7)
- added C46: 0.1μf, Capacitor_SMD:C_0201_0603Metric, B.Cu at (79.0, 65.6)
- added C47: 0.1μf, Capacitor_SMD:C_0201_0603Metric, B.Cu at (80.6, 74.2)
- added C48: 0.1μf, Capacitor_SMD:C_0201_0603Metric, B.Cu at (79.0, 76.1)
- C10, C11, C12, C13, C14, C15, C16, C17, C18, C19, C20, C21, C22, C23, C24, C25, C27, C28, C29, C30, C31, C32, C39, C5, C6, C7, C8, C9, R10: moved to B.Cu
- moved C8 29.0 mm to (80.5, 64.4)
- moved C7 27.4 mm to (82.4, 64.4)
- moved C28 26.4 mm to (79.0, 68.3), turned to 90 degrees
- moved C6 26.0 mm to (84.5, 64.4)
- moved C5 24.9 mm to (86.2, 64.4)
- moved C19 24.8 mm to (79.0, 69.6), turned to 90 degrees
- moved C20 22.8 mm to (80.2, 69.9), turned to 180 degrees
- moved R10 19.8 mm to (86.6, 73.6), turned to 180 degrees
- moved C21 17.5 mm to (85.8, 70.0), turned to 180 degrees
- moved C27 17.4 mm to (79.3, 71.9), turned to 0 degrees
- moved C18 17.2 mm to (82.1, 67.0), turned to 90 degrees
- moved C25 16.9 mm to (81.0, 71.9), turned to 0 degrees
- moved C14 16.9 mm to (82.1, 75.4)
- moved C9 16.3 mm to (86.2, 77.4), turned to -90 degrees
- moved C22 15.8 mm to (87.3, 70.0), turned to 180 degrees
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Routing:
- net DM0A: track 21.0 -> 0.00 mm, vias 2 -> 0
- net DQ4A: track 20.9 -> 0.00 mm, vias 2 -> 0
- net GND: track 60.7 -> 75.3 mm, vias 67 -> 93
- net +1V1: track 12.4 -> 18.6 mm, vias 1 -> 23
- net ZQ0: track 20.1 -> 18.7 mm, vias 3 -> 23
- net DQS0NA: track 21.0 -> 22.2 mm
- net +1V8: vias 1 -> 3
Other:
- board text added: "For Anahad: I left the 4.7uF capacitors out of the ways for now since I don't really know where to put them, uh.. may have placed some via in bad spots.."
- board text added: "Note: Most of the capacitors on the LPDDR4X have not been set correctly. It's the right capacitors, just the pins I/you must fix, and the traces.. Do not copy/paste the 4.7uF capacitors, may forget."
