File: stemthortyto/stemthortyto.kicad_sch (KiCad schematic)
At the start: 65 parts, among them IC1 E22-900M22S, J1 Jack-DC, Q1 BCV29, U1 LT1585-3.3, U2 ADXL343, U3 RK3588S, U4 K4UCE3Q4AB-MGCL, U5 FEMDRW032G-88A19

Commit message: Add files via upload
Parts:
- added C44, C46, C47: 0.1μf, Capacitor_SMD:C_0201_0603Metric, symbol Device:C_Small
Connections:
- net +0V6: now also C44.1, C46.1, C47.1
- net GND: now also C44.2, C46.2, C47.2
Other:
- moved on the sheet: C15, U3A, U3I, U3J
